File: kicad/AnalogSensors.sch (KiCad schematic (older format))
At the start: 8 parts, among them P201 Positive, P202 Negative

Commit message: More changes to the layout for the Power System integration
Parts:
- R201, R202: footprint Resistors_SMD:R_1206_HandSoldering -> Resistors_SMD:R_1206
- R203: footprint Resistors_SMD:R_0805_HandSoldering -> Resistors_SMD:R_0805
Changed lines of the file:
@@
 F 0 "R201" V 3580 1850 50  0000 C CNN
 F 1 "1MΩ 125mW  0.1%" H 4000 1800 50  0000 C CNN
-F 2 "Resistors_SMD:R_1206_HandSoldering" V 3430 1850 50  0001 C CNN
+F 2 "Resistors_SMD:R_1206" V 3430 1850 50  0001 C CNN
 F 3 "" H 3500 1850 50  0000 C CNN
 F 4 "SPR-1206 100K" H 3500 1850 60  0001 C CNN "MPN"
@@
 F 0 "R202" V 3580 2550 50  0000 C CNN
 F 1 "270kΩ 125mW  0.1%" H 4050 2500 50  0000 C CNN
-F 2 "Resistors_SMD:R_1206_HandSoldering" V 3430 2550 50  0001 C CNN
+F 2 "Resistors_SMD:R_1206" V 3430 2550 50  0001 C CNN
 F 3 "" H 3500 2550 50  0000 C CNN
 F 4 "SPR-1206 39,0K" H 3500 2550 60  0001 C CNN "MPN"
@@
 F 0 "R203" V 2530 2250 50  0000 C CNN
 F 1 "0Ω" V 2370 2250 50  0000 C CNN
-F 2 "Resistors_SMD:R_0805_HandSoldering" V 2380 2250 50  0001 C CNN
+F 2 "Resistors_SMD:R_0805" V 2380 2250 50  0001 C CNN
 F 3 "" H 2450 2250 50  0000 C CNN
 F 4 "Value" H 2450 2250 60  0001 C CNN "Link"
