File: kicad/FieldDevice.sch (KiCad schematic (older format))
At the start: 19 parts, among them U101 DS7505

Commit message: Reworking the schematic
Parts:
- removed C101: 100pF 50V, Capacitors_SMD:C_0805_HandSoldering, symbol C
- removed D101: Tx, Diodes_SMD:D_0805, symbol LED-RESCUE-FieldDevice
- removed D102: Rx, Diodes_SMD:D_0805, symbol LED-RESCUE-FieldDevice
- removed H102: DIGI_XBEE, FieldDevice_Footprints:XBEE_S2C, symbol DIGI_XBEE
- removed R104, R105, R106: 0, Resistors_SMD:R_0805_HandSoldering, symbol R
- removed R111: 10k, Resistors_SMD:R_0805_HandSoldering, symbol R
- removed R112, R113: 680Ω, Resistors_SMD:R_0805_HandSoldering, symbol R
- removed U101: DS7505, Housings_SOIC:SOIC-8_3.9x4.9mm_Pitch1.27mm, symbol DS7505
- added J?: Power IN, symbol Conn_01x02_Female
- added U?: Teensy-3.2, symbol Teensy-3.2
Connections:
- net labels added: 5V, I2C_SDA, Rx, SPI_CS, Vin
- net labels removed: CS, SDA
- wire segments 81 -> 53
- no-connect marks 16 -> 1
Other:
- note removed: "I²C Address '1010000'"
- note removed: "Temperature Sensor"
- note removed: "The minimal configuration \nfor the XBEE is Vcc, GND, \nDin and Dout"

Commit message: Completed the new schematic (draft) and started the layout to verify the design
Parts:
- removed H101: CE_Socket, CE_Header:CE_Socket, symbol CE_Header
- removed J?: Power IN, symbol Conn_01x02_Female
- removed R107, R108: 0Ω, Resistors_SMD:R_0805_HandSoldering, symbol R
- removed R109: 0, Resistors_SMD:R_0805_HandSoldering, symbol R
- removed R110: 4k7Ω, Resistors_SMD:R_0805_HandSoldering, symbol R
- added PWR101: FD_POWER, Pin_Headers:Pin_Header_Straight_1x03_Pitch2.54mm, symbol FD_POWER
- added R104: 0Ω, Resistors_SMD:R_0805_HandSoldering, symbol R
- added R105, R106: 4k7Ω, Resistors_SMD:R_0805_HandSoldering, symbol R
- R103: value 4k7Ω -> 0Ω
- U101: renamed from U?; footprint (none) -> FieldDevice_Footprints:Teensy-32
Connections:
- net labels added: BACKLIGHT
- net labels removed: RX, Vin
- wire segments 53 -> 48
- no-connect marks 1 -> 16
Other:
- note added: "The FD Power is a custom power module \nto deliver 5V and 3V3 from an input of\nbetween 6-18V\nThe initial physical connection will be \na 3 pole pin header."
- moved on the sheet: U101

Commit message: Completed the draft of REV2
Connections:
- net BACKLIGHT: now also U101.7 (7/RX3)
- no-connect marks 16 -> 15
Changed lines of the file:
@@
 EESchema Schematic File Version 2
-LIBS:FieldDevice-rescue
 LIBS:fieldDevice_symbols
 LIBS:ce_header
@@
 $EndComp
 Wire Wire Line
-	1750 2150 2200 2150
-Wire Wire Line
-	2200 2150 3150 2150
+	1750 2150 3150 2150
 Wire Wire Line
 	2200 2150 2200 2100
@@
 $EndComp
 Wire Wire Line
-	2350 2000 2750 2000
-Wire Wire Line
-	2750 2000 3150 2000
+	2350 2000 3150 2000
 Wire Wire Line
 	2750 2000 2750 1950
@@
 NoConn ~ 4950 1900
 NoConn ~ 4950 2050
-NoConn ~ 4950 2200
 NoConn ~ 3150 1700
 NoConn ~ 3150 1850
@@
 Wire Wire Line
 	2200 1800 2150 1800
+Text Label 5100 2200 0    60   ~ 0
+BACKLIGHT
+Wire Wire Line
+	4950 2200 5100 2200
 $EndSCHEMATC

Commit message: More changes to the layout for the Power System integration
Parts:
- PWR101: footprint Pin_Headers:Pin_Header_Straight_1x03_Pitch2.54mm -> Pin_Headers:Pin_Header_Angled_1x04_Pitch2.54mm
- R101, R102, R103, R104, R105, R106: footprint Resistors_SMD:R_0805_HandSoldering -> Resistors_SMD:R_0805
Connections:
- net 3V3: now also PWR101.2 (3V3); no longer PWR101.3 (BATT)
- net BACKLIGHT: now also U101.17 (17/A3); no longer U101.7 (7/RX3)
- net BATT: now reaches U101.2
- net BATT: now also PWR101.3 (BATT)
- no-connect marks 15 -> 14
Changed lines of the file:
@@
 Wire Wire Line
 	2100 4450 2300 4450
-Wire Wire Line
-	2100 4750 2300 4750
-Text Label 2300 4750 2    60   ~ 0
-3V3
 Text Label 2300 4450 2    60   ~ 0
 5V
@@
 Text Label 7600 4100 0    60   ~ 0
 BACKLIGHT
-$Comp
-L FD_POWER PWR101
-U 1 1 5A7391A5
-P 1200 4800
-F 0 "PWR101" H 1800 4650 60  0000 C CNN
-F 1 "FD_POWER" H 1550 5000 60  0000 C CNN
-F 2 "Pin_Headers:Pin_Header_Straight_1x03_Pitch2.54mm" H 1200 4800 60  0001 C CNN
-F 3 "" H 1200 4800 60  0001 C CNN
-	1    1200 4800
-	1    0    0    -1
-$EndComp
 Wire Wire Line
 	1550 5100 1550 5300
@@
 F 0 "R101" V 5280 1150 50  0000 C CNN
 F 1 "0Ω" V 5200 1150 50  0000 C CNN
-F 2 "Resistors_SMD:R_0805_HandSoldering" V 5130 1150 50  0001 C CNN
+F 2 "Resistors_SMD:R_0805" V 5130 1150 50  0001 C CNN
 F 3 "" H 5200 1150 50  0000 C CNN
 	1    5200 1150
@@
 F 0 "R102" V 5280 1300 50  0000 C CNN
 F 1 "0Ω" V 5200 1300 50  0000 C CNN
-F 2 "Resistors_SMD:R_0805_HandSoldering" V 5130 1300 50  0001 C CNN
+F 2 "Resistors_SMD:R_0805" V 5130 1300 50  0001 C CNN
 F 3 "" H 5200 1300 50  0000 C CNN
 	1    5200 1300
@@
 F 0 "R106" V 2280 1950 50  0000 C CNN
 F 1 "4k7Ω" V 2200 1950 50  0000 C CNN
-F 2 "Resistors_SMD:R_0805_HandSoldering" V 2130 1950 50  0001 C CNN
+F 2 "Resistors_SMD:R_0805" V 2130 1950 50  0001 C CNN
 F 3 "" H 2200 1950 50  0000 C CNN
 	1    2200 1950
@@
 F 0 "R105" V 2830 1800 50  0000 C CNN
 F 1 "4k7Ω" V 2750 1800 50  0000 C CNN
-F 2 "Resistors_SMD:R_0805_HandSoldering" V 2680 1800 50  0001 C CNN
+F 2 "Resistors_SMD:R_0805" V 2680 1800 50  0001 C CNN
 F 3 "" H 2750 1800 50  0000 C CNN
 	1    2750 1800
@@
 F 0 "R103" V 2980 1400 50  0000 C CNN
 F 1 "0Ω" V 2900 1400 50  0000 C CNN
-F 2 "Resistors_SMD:R_0805_HandSoldering" V 2830 1400 50  0001 C CNN
+F 2 "Resistors_SMD:R_0805" V 2830 1400 50  0001 C CNN
 F 3 "" H 2900 1400 50  0000 C CNN
 	1    2900 1400
@@
 F 0 "R104" V 2980 1550 50  0000 C CNN
 F 1 "0Ω" V 2900 1550 50  0000 C CNN
-F 2 "Resistors_SMD:R_0805_HandSoldering" V 2830 1550 50  0001 C CNN
+F 2 "Resistors_SMD:R_0805" V 2830 1550 50  0001 C CNN
 F 3 "" H 2900 1550 50  0000 C CNN
 	1    2900 1550
@@
 Wire Wire Line
 	3050 1550 3150 1550
-NoConn ~ 4950 1450
 NoConn ~ 4950 1600
 NoConn ~ 4950 1750
@@
 NoConn ~ 3150 1700
 NoConn ~ 3150 1850
-NoConn ~ 3150 2300
+NoConn ~ 4950 2200
 NoConn ~ 3150 2450
 NoConn ~ 3150 2600
@@
 Wire Wire Line
 	2200 1800 2150 1800
-Text Label 5100 2200 0    60   ~ 0
+Text Label 2950 2300 2    60   ~ 0
 BACKLIGHT
 Wire Wire Line
-	4950 2200 5100 2200
+	3150 2300 2950 2300
+$Comp
+L FD_POWER PWR101
+U 1 1 5A75CF63
+P 1200 4800
+F 0 "PWR101" H 1800 4650 60  0000 C CNN
+F 1 "FD_POWER" H 1550 5000 60  0000 C CNN
+F 2 "Pin_Headers:Pin_Header_Angled_1x04_Pitch2.54mm" H 1200 4800 60  0001 C CNN
+F 3 "" H 1200 4800 60  0001 C CNN
+	1    1200 4800
+	1    0    0    -1
+$EndComp
+Wire Wire Line
+	2100 4550 2300 4550
+Text Label 2300 4550 2    60   ~ 0
+3V3
+Wire Wire Line
+	2100 4750 2300 4750
+Text Label 2300 4750 2    60   ~ 0
+BATT
+Text Label 5600 1450 2    60   ~ 0
+BATT
+Wire Wire Line
+	4950 1450 5600 1450
 $EndSCHEMATC
