File: kicad/TemperatureSensor.sch (KiCad schematic (older format))
At the start: 6 parts

Commit message: Completed the new schematic (draft) and started the layout to verify the design
Parts:
- gave numbers to parts that had none: 6
Other:
- note added: "The purpose of this temperature unit\nis to measure and report the temperature\nof the Field Device board. This is not \nintended as any type of environmental\nsensor other than device running conditions.\n"
Changed lines of the file:
@@
 $Descr A4 11693 8268
 encoding utf-8
-Sheet 6 6
+Sheet 5 5
 Title ""
 Date ""
@@
 $EndDescr
 $Comp
-L DS7505 U?
+L DS7505 U501
 U 1 1 5A7136A0
 P 4600 3200
-F 0 "U?" H 4950 2750 60  0000 C CNN
+F 0 "U501" H 4950 2750 60  0000 C CNN
 F 1 "DS7505" H 4600 3550 60  0000 C CNN
 F 2 "Housings_SOIC:SOIC-8_3.9x4.9mm_Pitch1.27mm" H 4600 3000 60  0001 C CNN
@@
 3V3
 $Comp
-L GND #PWR?
+L GND #PWR010
 U 1 1 5A7136A8
 P 3650 3700
-F 0 "#PWR?" H 3650 3450 50  0001 C CNN
+F 0 "#PWR010" H 3650 3450 50  0001 C CNN
 F 1 "GND" H 3650 3550 50  0000 C CNN
 F 2 "" H 3650 3700 50  0000 C CNN
@@
 $EndComp
 $Comp
-L R R?
+L R R502
 U 1 1 5A7136AE
 P 5450 3850
-F 0 "R?" V 5530 3850 50  0000 C CNN
+F 0 "R502" V 5530 3850 50  0000 C CNN
 F 1 "0" V 5450 3850 50  0000 C CNN
 F 2 "Resistors_SMD:R_0805_HandSoldering" V 5380 3850 50  0001 C CNN
@@
 $EndComp
 $Comp
-L R R?
+L R R503
 U 1 1 5A7136B5
 P 5700 3850
-F 0 "R?" V 5780 3850 50  0000 C CNN
+F 0 "R503" V 5780 3850 50  0000 C CNN
 F 1 "0" V 5700 3850 50  0000 C CNN
 F 2 "Resistors_SMD:R_0805_HandSoldering" V 5630 3850 50  0001 C CNN
@@
 $EndComp
 $Comp
-L R R?
+L R R504
 U 1 1 5A7136BC
 P 5950 3850
-F 0 "R?" V 6030 3850 50  0000 C CNN
+F 0 "R504" V 6030 3850 50  0000 C CNN
 F 1 "0" V 5950 3850 50  0000 C CNN
 F 2 "Resistors_SMD:R_0805_HandSoldering" V 5880 3850 50  0001 C CNN
@@
 $EndComp
 $Comp
-L GND #PWR?
+L GND #PWR011
 U 1 1 5A7136C3
 P 5550 4250
-F 0 "#PWR?" H 5550 4000 50  0001 C CNN
+F 0 "#PWR011" H 5550 4000 50  0001 C CNN
 F 1 "GND" H 5550 4100 50  0000 C CNN
 F 2 "" H 5550 4250 50  0000 C CNN
@@
 OverTemp
 Wire Wire Line
-	5250 2900 6250 2900
-Wire Wire Line
-	6250 2900 6550 2900
+	5250 2900 6550 2900
 Wire Wire Line
 	3900 3500 3650 3500
@@
 	3900 3100 3450 3100
 Wire Wire Line
-	2050 3300 2600 3300
-Wire Wire Line
-	2600 3300 3900 3300
+	2050 3300 3900 3300
 Wire Wire Line
 	5450 4000 5450 4150
 Wire Wire Line
-	5450 4150 5550 4150
-Wire Wire Line
-	5550 4150 5700 4150
-Wire Wire Line
-	5700 4150 5950 4150
+	5450 4150 5950 4150
 Wire Wire Line
 	5950 4150 5950 4000
@@
 	5950 3100 5950 3700
 $Comp
-L R R?
+L R R501
 U 1 1 5A7136E1
 P 2600 2600
-F 0 "R?" V 2680 2600 50  0000 C CNN
+F 0 "R501" V 2680 2600 50  0000 C CNN
 F 1 "10k" V 2600 2600 50  0000 C CNN
 F 2 "Resistors_SMD:R_0805_HandSoldering" V 2530 2600 50  0001 C CNN
@@
 	6250 2900 6250 3000
 $Comp
-L C C?
+L C C501
 U 1 1 5A7136EE
 P 6250 3150
-F 0 "C?" H 6275 3250 50  0000 L CNN
+F 0 "C501" H 6275 3250 50  0000 L CNN
 F 1 "100pF 50V" H 6275 3050 50  0000 L CNN
 F 2 "Capacitors_SMD:C_0805_HandSoldering" H 6288 3000 30  0001 C CNN
@@
 $EndComp
 $Comp
-L GND #PWR?
+L GND #PWR012
 U 1 1 5A7136F5
 P 6250 3400
-F 0 "#PWR?" H 6250 3150 50  0001 C CNN
+F 0 "#PWR012" H 6250 3150 50  0001 C CNN
 F 1 "GND" H 6250 3250 50  0000 C CNN
 F 2 "" H 6250 3400 50  0000 C CNN
@@
 Text HLabel 3450 3100 0    60   Input ~ 0
 I2C_SCK
+Text Notes 3700 5150 0    60   ~ 0
+The purpose of this temperature unit\nis to measure and report the temperature\nof the Field Device board. This is not \nintended as any type of environmental\nsensor other than device running conditions.\n
 $EndSCHEMATC

Commit message: Completed the draft of REV2
Connections:
- net A2: now reaches R502.1, U501.5 (A2)
- net A1: now reaches R503.1, U501.6 (A1)
- net A0: now reaches R504.1, U501.7 (A0)
Changed lines of the file:
@@
 EESchema Schematic File Version 2
-LIBS:FieldDevice-rescue
 LIBS:fieldDevice_symbols
 LIBS:ce_header
@@
 Text Notes 3700 5150 0    60   ~ 0
 The purpose of this temperature unit\nis to measure and report the temperature\nof the Field Device board. This is not \nintended as any type of environmental\nsensor other than device running conditions.\n
+Text Label 5300 3500 0    60   ~ 0
+A2
+Text Label 5300 3300 0    60   ~ 0
+A1
+Text Label 5300 3100 0    60   ~ 0
+A0
 $EndSCHEMATC

Commit message: More changes to the layout for the Power System integration
Parts:
- C501: footprint Capacitors_SMD:C_0805_HandSoldering -> Capacitors_SMD:C_0805
- R501, R502, R503, R504: footprint Resistors_SMD:R_0805_HandSoldering -> Resistors_SMD:R_0805
Changed lines of the file:
@@
 F 0 "R502" V 5530 3850 50  0000 C CNN
 F 1 "0" V 5450 3850 50  0000 C CNN
-F 2 "Resistors_SMD:R_0805_HandSoldering" V 5380 3850 50  0001 C CNN
+F 2 "Resistors_SMD:R_0805" V 5380 3850 50  0001 C CNN
 F 3 "" H 5450 3850 50  0000 C CNN
 	1    5450 3850
@@
 F 0 "R503" V 5780 3850 50  0000 C CNN
 F 1 "0" V 5700 3850 50  0000 C CNN
-F 2 "Resistors_SMD:R_0805_HandSoldering" V 5630 3850 50  0001 C CNN
+F 2 "Resistors_SMD:R_0805" V 5630 3850 50  0001 C CNN
 F 3 "" H 5700 3850 50  0000 C CNN
 	1    5700 3850
@@
 F 0 "R504" V 6030 3850 50  0000 C CNN
 F 1 "0" V 5950 3850 50  0000 C CNN
-F 2 "Resistors_SMD:R_0805_HandSoldering" V 5880 3850 50  0001 C CNN
+F 2 "Resistors_SMD:R_0805" V 5880 3850 50  0001 C CNN
 F 3 "" H 5950 3850 50  0000 C CNN
 	1    5950 3850
@@
 F 0 "R501" V 2680 2600 50  0000 C CNN
 F 1 "10k" V 2600 2600 50  0000 C CNN
-F 2 "Resistors_SMD:R_0805_HandSoldering" V 2530 2600 50  0001 C CNN
+F 2 "Resistors_SMD:R_0805" V 2530 2600 50  0001 C CNN
 F 3 "" H 2600 2600 50  0000 C CNN
 	1    2600 2600
@@
 F 0 "C501" H 6275 3250 50  0000 L CNN
 F 1 "100pF 50V" H 6275 3050 50  0000 L CNN
-F 2 "Capacitors_SMD:C_0805_HandSoldering" H 6288 3000 30  0001 C CNN
+F 2 "Capacitors_SMD:C_0805" H 6288 3000 30  0001 C CNN
 F 3 "" H 6250 3150 60  0000 C CNN
 F 4 "Value" H 6250 3150 60  0001 C CNN "Link"
